File: Schematics/RGBW-Lampe/RGBW-Lampe Control.sch (KiCad schematic (older format))
At the start: 74 parts, among them J1 Conn_01x10, J2 Conn_01x04, J5 Conn_01x04_Male, J6 Conn_02x05_Odd_Even, J8 Conn_01x02, Q1 BSS138, Q2 BSS138, Q3 BSS138, Q4 BSS138, T1 SFH320, U1 LIS2DH, U2 ESP-12F, U4 24LC16, U5 TSOP348xx, U7 STM32L151CBTx, Y1 12MHz, Y2 32,768 MS1V 7

Commit message: PCB version produced
Parts:
- removed C37: 220n, Capacitor_SMD:C_0603_1608Metric, symbol Device:C
- removed J2: Conn_01x04, Connector_Stocko:Stocko_MKS_1654-6-0-404_1x4_P2.50mm_Vertical, symbol Connector_Generic:Conn_01x04
- removed J8: Conn_01x02, Connector_Stocko:Stocko_MKS_1652-6-0-202_1x2_P2.50mm_Vertical, symbol Connector_Generic:Conn_01x02
- removed R16: 100, Resistor_SMD:R_0805_2012Metric, symbol Device:R
- added C54, C55, C56: 10n, Capacitor_SMD:C_0603_1608Metric, symbol Device:C
- added J9: Conn_02x05_Odd_Even, Connector_IDC:IDC-Header_2x05_P2.54mm_Vertical, symbol Connector_Generic:Conn_02x05_Odd_Even
- added JP2, JP3, JP4: Jumper_3_Open, Connector_PinHeader_2.54mm:PinHeader_1x03_P2.54mm_Vertical, symbol Jumper:Jumper_3_Open
- added JP5, JP6: Jumper_2_Open, Connector_PinHeader_2.54mm:PinHeader_1x02_P2.54mm_Vertical, symbol Jumper:Jumper_2_Open
- added JP7, JP8: SolderJumper_2_Open, Jumper:SolderJumper-2_P1.3mm_Open_Pad1.0x1.5mm, symbol Jumper:SolderJumper_2_Open
- added R42: 10k, Resistor_SMD:R_0805_2012Metric, symbol Device:R
- added R45, R46, R47: ob, Resistor_SMD:R_0805_2012Metric, symbol Device:R
- L7, L8: value BLM18 -> BLM21PG 331
- R35, R36: value 10k -> 4,7k
Connections:
- net LCD_Backlight_PWM is gone; now on net LCD_BACKLIGHT_PWM: U7.19 (PB1)
- net +12V: now also R45.1, R46.1, R47.1; no longer C1.1, R3.2
- net +3V3: now also C1.1, R3.2, U7.1 (VLCD), C54.1, C55.1, J9.3 (Pin_3)
- net ESP_RST: now also R29.1; no longer U2.1 (~RST)
- net GND: now also C54.2, C55.2, C56.2, J9.1 (Pin_1), J9.2 (Pin_2), J9.5 (Pin_5), J9.7 (Pin_7), JP5.2 (B), JP6.2 (B)
- net SCL: now also JP7.2 (B)
- net SDA: now also JP8.2 (B)
- net ExtPower: now reaches U2.6 (GPIO12)
- net at C28.1, C30.1, L8.2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: now also C56.1, R42.1
- net at LED1.4 (C), R2.1: now also R46.2
- net at LED1.6 (C), R1.1: now also R45.2
- net at C31.1, R19.1, R26.2: now also J9.4 (Pin_4)
- net at C33.1, R20.1: now also J9.9 (Pin_9)
- net at C32.1, R21.1: now also J9.10 (Pin_10)
- net at LED1.5 (C), R4.1: now also R47.2
- net at R29.2: now also U2.1 (~RST), JP5.1 (A); no longer J1.2 (Pin_2)
- net ESP_GPIO_0: no longer names the net of U2.18 (GPIO0)
- net ESP_GPIO_0: now also JP6.1 (A), R42.2; no longer U7.2 (PC13)
- removed net USART1_RX: R29.1, U2.22 (GPIO1/TXD), U7.31 (PA10)
- removed net USART1_TX: J1.9 (Pin_9), U2.21 (GPIO3/RXD), U7.30 (PA9)
- new net: J9.8 (Pin_8), JP7.1 (A)
- new net: J9.6 (Pin_6), JP8.1 (A)
- new net AMP_SHTDN: U7.2 (PC13)
- new net ESP_RX: JP4.2 (C), U2.21 (GPIO3/RXD)
- new net ESP_TX: JP2.1 (A), JP3.1 (A), U2.22 (GPIO1/TXD)
- new net J-Link_RX: J1.9 (Pin_9), JP2.2 (C)
- new net J-Link_TX: J1.2 (Pin_2), JP3.3 (B), JP4.3 (B)
- new net STM32_RX: JP3.2 (C), U7.31 (PA10)
- new net STM32_TX: JP2.3 (B), JP4.1 (A), U7.30 (PA9)
Other:
- note added: "Close to Progam ESP"
- note added: "Close to force\nESP reset"
- moved on the sheet: L8, LED1A, LED1B, LED1C, R1, R2, R34, R4
