File: Schematics/RGBW-Lampe/RGBW-Lampe Power.sch (KiCad schematic (older format))
At the start: 68 parts, among them J3 Conn_01x08, J4 Conn_01x02, J7 Conn_01x02, U3 L5973D, U6 TDA7052A

Commit message: PCB version produced
Parts:
- removed C47: 220nF / 25V, Capacitor_SMD:C_0603_1608Metric, symbol Device:C
- removed C49: 470µF / 25V, Capacitor_THT:CP_Radial_D8.0mm_P3.50mm, symbol Device:CP
- removed U6: TDA7052A, Package_SO:SO-8_3.9x4.9mm_P1.27mm, symbol Amplifier_Audio:TDA7052A
- added C37: 1µF / 50V X7R, Capacitor_SMD:C_1206_3216Metric, symbol Device:C
- added C47: 100µF / 6,3V, Capacitor_SMD:C_1206_3216Metric, symbol RGBW-Lampe-eagle-import:C-EUC0805
- added C49: 1n, Capacitor_SMD:C_0603_1608Metric, symbol Device:C
- added C53: 220nF / 25V, Capacitor_SMD:C_0603_1608Metric, symbol Device:C
- added C57, C58: 10n, Capacitor_SMD:C_0603_1608Metric, symbol Device:C
- added J8: Conn_01x02, Connector_JST:JST_XH_B2B-XH-A_1x02_P2.50mm_Vertical, symbol Connector_Generic:Conn_01x02
- added R16: 22k, Resistor_SMD:R_0805_2012Metric, symbol Device:R
- added R43: 180, Resistor_SMD:R_0805_2012Metric, symbol Device:R
- added R44: 1.2k, Resistor_SMD:R_0805_2012Metric, symbol Device:R
- added U6: LM4861M, LM4861:LM4861M, symbol LM4861:LM4861M
- added U8: ISP762T, ISP762:ISP762T, symbol ISP762:ISP762T
- J3: footprint Connector_Stocko:Stocko_MKS_1658-6-0-808_1x8_P2.50mm_Vertical -> Connector_JST:JST_XH_B8B-XH-A_1x08_P2.50mm_Vertical
- J4, J7: footprint Connector_Stocko:Stocko_MKS_1652-6-0-202_1x2_P2.50mm_Vertical -> Connector_JST:JST_XH_B2B-XH-A_1x02_P2.50mm_Vertical
- R10, R11, R7, R8: value 0.2 -> 0.150
- R37: value 100 -> 22k
- R38: value 100 -> 1.2k
Connections:
- net +12V: now also C53.2, U8.5 (VBB), U8.6 (VBB), U8.7 (VBB), U8.8 (VBB)
- net +12VA: no longer L9.1
- net +3V3: now also L9.1, C57.2
- net GND: now also C48.1, D6.2 (A), C37.2, C47.2, C53.1, C57.1, C58.1, J8.1 (Pin_1), R44.1, U6.7 (GND), U8.1 (GND); no longer D6.1 (K)
- net LED_1_PWM: now also R32.1; no longer R22.1
- net LED_2_PWM: now also R33.1; no longer R23.1
- net LED_3_PWM: now also R22.1; no longer R32.1
- net LED_4_PWM: now also R23.1; no longer R33.1
- net Volume: now also R43.2; no longer R37.2
- net at L6.P$1, U3.1 (OUT): now also D6.1 (K); no longer D6.2 (A)
- net at C48.2, L9.2: now also C47.1, C58.2, U6.6 (VDD)
- net at C46.1: now also R37.2
- net at R37.1: now also C49.1, R16.2, U6.4 (-IN)
- net at J7.1 (Pin_1): now also U6.8 (VO2)
- net at J7.2 (Pin_2): now also C49.2, R16.1, U6.5 (VO1)
- net at C46.2, C50.2, R38.1: now also R43.1, R44.2
- new net: C37.1, U6.2 (BYPASS), U6.3 (+IN)
- new net: J8.2 (Pin_2), U8.3 (OUT)
- new net AMP_SHTDN: U6.1 (SHTDN)
- new net ExtPower: U8.2 (IN)
Other:
- note added: "666mA per Driver"
- note added: "Changes for 1A per driver\nInductor 242418 FPS 47µH\nR 0.100 Ohm\nDiode MBRS 240 SMD"
- moved on the sheet: C46, C48, C50, H1, H2, H3, H4, J7, L9, R37, R38
